File: hardware/duinolpcfwhspi.brd (EAGLE design)
At the start: 53.3 x 45.8 mm, 27 parts

Commit message: hardware documentation: add schematic i just hacked together
Parts:
- removed ANALOG1, J7: (no value), pinhead:1X06
- added DIGI_DN, DIGI_UP: (no value), SmartPrj:1X08-TH
- J1, POWER: device SmartPrj:1X08-TH -> pinhead:1X06
- PLCC32: value (none) -> PLCC32
- RESET: value B2 -> (none)
- moved POWER 48.7 mm to (2.54, 26.7)
- moved J1 48.2 mm to (5.08, 26.7), turned to 270 degrees
- renumbered E$11 to R3, E$12 to R2, E$14 to R4, E$16 to R5, E$18 to R9, E$2 to R10, E$20 to R8, E$21 to R7, E$24 to R6, E$25 to C1, E$3 to R15, E$4 to R14, E$5 to R11, E$7 to R13, E$8 to R12, E$9 to R1, J5 to J4, J6 to J3, POWER1 to J2, S2 to RESET
Connections:
- net N$13 renamed LPCD0
- net N$14 renamed LPCD1
- net N$15 renamed LPCD2
- net N$39 renamed LPCD3
- net S$1 renamed PC5
- net S$2 renamed PC4
- removed net N$16: J1.1, J4.1
- removed net N$29: J1.2, J4.2
- removed net N$34: J1.6, J4.6
- removed net N$35: J1.7, J4.7
- removed net S$10: ANALOG1.6, J7.6
- removed net S$12: ANALOG1.3, J7.3
- removed net S$13: ANALOG1.1, J7.1, RESET.2
- removed net S$24: J2.3, POWER.3, R4.2
- removed net S$26: J2.5, POWER.5, R2.2
- removed net S$7: J2.1, POWER.1
- removed net S$8: J2.6, POWER.6
- removed net S$9: J2.7, POWER.7
- new net 5V0: J1.3, POWER.3
- new net AREF: DIGI_UP.1, J2.1
- new net HSCLK: DIGI_UP.3, J2.3, R4.2
- new net HSDI: DIGI_UP.5, J2.5, R2.2
- new net PB1: DIGI_UP.7, J2.7
- new net PB2: DIGI_UP.6, J2.6
- new net PD0: DIGI_DN.1, J4.1
- new net PD1: DIGI_DN.2, J4.2
- new net PD5: DIGI_DN.6, J4.6
- new net PD6: DIGI_DN.7, J4.7
- new net RESET: J1.1, POWER.1, RESET.2
- new net VIN: J1.6, POWER.6
- net 3V3: now also J1.2, POWER.2; no longer ANALOG1.2, J7.2
- net FRAME: now also DIGI_DN.4; no longer J1.4
- net GND: now also DIGI_UP.2, J1.4, J1.5, POWER.4, POWER.5; no longer ANALOG1.4, ANALOG1.5, J7.4, J7.5, POWER.2
- net INIT: now also DIGI_DN.5; no longer J1.5
- net LCLK: now also DIGI_DN.8; no longer J1.8
- net LRST: now also DIGI_DN.3; no longer J1.3
- net SCS: now also DIGI_UP.8; no longer POWER.8
- net SDO: now also DIGI_UP.4; no longer POWER.4
Routing:
- net S$26: track 18.8 -> 0.00 mm
- net HSDI: track 0.00 -> 18.8 mm
- net S$24: track 12.0 -> 0.00 mm
- net HSCLK: track 0.00 -> 12.0 mm
- net S$13: track 10.0 -> 0.00 mm
- net RESET: track 0.00 -> 10.0 mm
- net VIN: track 0.00 -> 2.54 mm
- net S$12: track 2.54 -> 0.00 mm
- net S$10: track 2.54 -> 0.00 mm
- net 5V0: track 0.00 -> 2.54 mm
- net S$9: track 2.54 -> 0.00 mm
- net S$8: track 2.54 -> 0.00 mm
- net S$7: track 2.54 -> 0.00 mm
- net PD6: track 0.00 -> 2.54 mm
- net PD5: track 0.00 -> 2.54 mm
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